Commit message: minor changes

File: models/cylinder.urdf (robot description, URDF)
Before this commit: robot cylinder, 1 links, 0 joints
Links:
- link base_link: geometry visual cylinder length=2.0 radius=0.02

Commit message: minor changes

File: models/cylinder.urdf (robot description, URDF)
Before this commit: robot cylinder, 1 links, 0 joints
Links:
- link base_link: geometry visual cylinder length=2.0 radius=0.1
